Commit message: Single iiwa simulation setup and working with position based controllers, moveit configuration has been setup and works

File: iiwa_fri_description/urdf/dual_iiwa.urdf.xacro (robot description, xacro)
@@ -2,8 +2,8 @@
 <robot xmlns:xacro="http://www.ros.org/wiki/xacro" name="dual_iiwa">
   <!-- Import Rviz colors -->
-  <xacro:include filename="$(find sat_iiwa_description)/urdf/materials.xacro" />
+  <xacro:include filename="$(find iiwa_fri_description)/urdf/materials.xacro" />
   <!--Import the iiwa macros -->
-  <xacro:include filename="$(find sat_iiwa_description)/urdf/iiwa14.xacro"/>
-  <xacro:include filename="$(find sat_iiwa_description)/urdf/iiwa7.xacro"/>
+  <xacro:include filename="$(find iiwa_fri_description)/urdf/iiwa14.xacro"/>
+  <xacro:include filename="$(find iiwa_fri_description)/urdf/iiwa7.xacro"/>
   <!--  Hardware interface options (currently both robots will need the same interface -->
   <xacro:arg name="hardware_interface" default="PositionJointInterface"/>

File: iiwa_fri_description/urdf/iiwa14.urdf.xacro (robot description, xacro)
@@ -2,7 +2,7 @@
 <robot name="iiwa14" xmlns:xacro="http://www.ros.org/wiki/xacro">
   <!-- Import Rviz colors -->
-  <xacro:include filename="$(find sat_iiwa_description)/urdf/materials.xacro" />
+  <xacro:include filename="$(find iiwa_fri_description)/urdf/materials.xacro" />
   <!--Import the lbr iiwa macro -->
-  <xacro:include filename="$(find sat_iiwa_description)/urdf/iiwa14.xacro"/>
+  <xacro:include filename="$(find iiwa_fri_description)/urdf/iiwa14.xacro"/>
   <xacro:arg name="hardware_interface" default="PositionJointInterface"/>
   <xacro:arg name="robot_name" default="iiwa14"/>

File: iiwa_fri_description/urdf/iiwa14.xacro (robot description, xacro)
@@ -2,9 +2,9 @@
 <robot xmlns:xacro="http://www.ros.org/wiki/xacro">
   <!-- Import all Gazebo-customization elements, including Gazebo colors -->
-  <xacro:include filename="$(find iiwa_description)/urdf/iiwa.gazebo.xacro" />
+  <xacro:include filename="$(find iiwa_fri_description)/urdf/iiwa.gazebo.xacro" />
   <!-- Import Transmissions -->
-  <xacro:include filename="$(find iiwa_description)/urdf/iiwa.transmission.xacro" />
+  <xacro:include filename="$(find iiwa_fri_description)/urdf/iiwa.transmission.xacro" />
   <!-- Include Utilities -->
-  <xacro:include filename="$(find iiwa_description)/urdf/utilities.xacro" />
+  <xacro:include filename="$(find iiwa_fri_description)/urdf/utilities.xacro" />
   <!-- some constants -->
   <xacro:property name="safety_controller_k_pos" value="100" />
@@ -29,5 +29,5 @@
         <origin xyz="0 0 0" rpy="0 0 0"/>
         <geometry>
-          <mesh filename="package://iiwa_description/meshes/iiwa14/visual/link_0.stl"/>
+          <mesh filename="package://iiwa_fri_description/meshes/iiwa14/visual/link_0.stl"/>
         </geometry>
         <material name="Grey"/>
@@ -36,5 +36,5 @@
         <origin xyz="0 0 0" rpy="0 0 0"/>
         <geometry>
-          <mesh filename="package://iiwa_description/meshes/iiwa14/collision/link_0.stl"/>
+          <mesh filename="package://iiwa_fri_description/meshes/iiwa14/collision/link_0.stl"/>
         </geometry>
         <material name="Grey"/>
@@ -70,12 +70,12 @@
         <origin xyz="0 0 0" rpy="0 0 0"/>
         <geometry>
-          <mesh filename="package://iiwa_description/meshes/iiwa14/visual/link_1.stl"/>
-        </geometry>
-        <material name="Orange"/>
-      </visual>
-      <collision>
-        <origin xyz="0 0 0" rpy="0 0 0"/>
-        <geometry>
-          <mesh filename="package://iiwa_description/meshes/iiwa14/collision/link_1.stl"/>
+          <mesh filename="package://iiwa_fri_description/meshes/iiwa14/visual/link_1.stl"/>
+        </geometry>
+        <material name="Orange"/>
+      </visual>
+      <collision>
+        <origin xyz="0 0 0" rpy="0 0 0"/>
+        <geometry>
+          <mesh filename="package://iiwa_fri_description/meshes/iiwa14/collision/link_1.stl"/>
         </geometry>
         <material name="Orange"/>
@@ -105,12 +105,12 @@
         <origin xyz="0 0 0" rpy="0 0 0"/>
         <geometry>
-          <mesh filename="package://iiwa_description/meshes/iiwa14/visual/link_2.stl"/>
-        </geometry>
-        <material name="Orange"/>
-      </visual>
-      <collision>
-        <origin xyz="0 0 0" rpy="0 0 0"/>
-        <geometry>
-          <mesh filename="package://iiwa_description/meshes/iiwa14/collision/link_2.stl"/>
+          <mesh filename="package://iiwa_fri_description/meshes/iiwa14/visual/link_2.stl"/>
+        </geometry>
+        <material name="Orange"/>
+      </visual>
+      <collision>
+        <origin xyz="0 0 0" rpy="0 0 0"/>
+        <geometry>
+          <mesh filename="package://iiwa_fri_description/meshes/iiwa14/collision/link_2.stl"/>
         </geometry>
         <material name="Orange"/>
@@ -140,12 +140,12 @@
         <origin xyz="0 0 0" rpy="0 0 0"/>
         <geometry>
-          <mesh filename="package://iiwa_description/meshes/iiwa14/visual/link_3.stl"/>
-        </geometry>
-        <material name="Orange"/>
-      </visual>
-      <collision>
-        <origin xyz="0 0 0" rpy="0 0 0"/>
-        <geometry>
-          <mesh filename="package://iiwa_description/meshes/iiwa14/collision/link_3.stl"/>
+          <mesh filename="package://iiwa_fri_description/meshes/iiwa14/visual/link_3.stl"/>
+        </geometry>
+        <material name="Orange"/>
+      </visual>
+      <collision>
+        <origin xyz="0 0 0" rpy="0 0 0"/>
+        <geometry>
+          <mesh filename="package://iiwa_fri_description/meshes/iiwa14/collision/link_3.stl"/>
         </geometry>
         <material name="Orange"/>
@@ -175,12 +175,12 @@
         <origin xyz="0 0 0" rpy="0 0 0"/>
         <geometry>
-          <mesh filename="package://iiwa_description/meshes/iiwa14/visual/link_4.stl"/>
-        </geometry>
-        <material name="Orange"/>
-      </visual>
-      <collision>
-        <origin xyz="0 0 0" rpy="0 0 0"/>
-        <geometry>
-          <mesh filename="package://iiwa_description/meshes/iiwa14/collision/link_4.stl"/>
+          <mesh filename="package://iiwa_fri_description/meshes/iiwa14/visual/link_4.stl"/>
+        </geometry>
+        <material name="Orange"/>
+      </visual>
+      <collision>
+        <origin xyz="0 0 0" rpy="0 0 0"/>
+        <geometry>
+          <mesh filename="package://iiwa_fri_description/meshes/iiwa14/collision/link_4.stl"/>
         </geometry>
         <material name="Orange"/>
@@ -210,12 +210,12 @@
         <origin xyz="0 0 0" rpy="0 0 0"/>
         <geometry>
-          <mesh filename="package://iiwa_description/meshes/iiwa14/visual/link_5.stl"/>
-        </geometry>
-        <material name="Orange"/>
-      </visual>
-      <collision>
-        <origin xyz="0 0 0" rpy="0 0 0"/>
-        <geometry>
-          <mesh filename="package://iiwa_description/meshes/iiwa14/collision/link_5.stl"/>
+          <mesh filename="package://iiwa_fri_description/meshes/iiwa14/visual/link_5.stl"/>
+        </geometry>
+        <material name="Orange"/>
+      </visual>
+      <collision>
+        <origin xyz="0 0 0" rpy="0 0 0"/>
+        <geometry>
+          <mesh filename="package://iiwa_fri_description/meshes/iiwa14/collision/link_5.stl"/>
         </geometry>
         <material name="Orange"/>
@@ -245,12 +245,12 @@
         <origin xyz="0 0 0" rpy="0 0 0"/>
         <geometry>
-          <mesh filename="package://iiwa_description/meshes/iiwa14/visual/link_6.stl"/>
-        </geometry>
-        <material name="Orange"/>
-      </visual>
-      <collision>
-        <origin xyz="0 0 0" rpy="0 0 0"/>
-        <geometry>
-          <mesh filename="package://iiwa_description/meshes/iiwa14/collision/link_6.stl"/>
+          <mesh filename="package://iiwa_fri_description/meshes/iiwa14/visual/link_6.stl"/>
+        </geometry>
+        <material name="Orange"/>
+      </visual>
+      <collision>
+        <origin xyz="0 0 0" rpy="0 0 0"/>
+        <geometry>
+          <mesh filename="package://iiwa_fri_description/meshes/iiwa14/collision/link_6.stl"/>
         </geometry>
         <material name="Orange"/>
@@ -280,5 +280,5 @@
         <origin xyz="0 0 0" rpy="0 0 0"/>
         <geometry>
-          <mesh filename="package://iiwa_description/meshes/iiwa14/visual/link_7.stl"/>
+          <mesh filename="package://iiwa_fri_description/meshes/iiwa14/visual/link_7.stl"/>
         </geometry>
         <material name="Grey"/>
@@ -287,5 +287,5 @@
         <origin xyz="0 0 0" rpy="0 0 0"/>
         <geometry>
-          <mesh filename="package://iiwa_description/meshes/iiwa14/collision/link_7.stl"/>
+          <mesh filename="package://iiwa_fri_description/meshes/iiwa14/collision/link_7.stl"/>
         </geometry>
         <material name="Grey"/>

File: iiwa_fri_description/urdf/iiwa7.urdf.xacro (robot description, xacro)
@@ -2,7 +2,7 @@
 <robot name="iiwa7" xmlns:xacro="http://www.ros.org/wiki/xacro">
   <!-- Import Rviz colors -->
-  <xacro:include filename="$(find iiwa_description)/urdf/materials.xacro" />
+  <xacro:include filename="$(find iiwa_fri_description)/urdf/materials.xacro" />
   <!--Import the lbr iiwa macro -->
-  <xacro:include filename="$(find iiwa_description)/urdf/iiwa7.xacro"/>
+  <xacro:include filename="$(find iiwa_fri_description)/urdf/iiwa7.xacro"/>
   <xacro:arg name="hardware_interface" default="PositionJointInterface"/>
   <xacro:arg name="robot_name" default="iiwa7"/>

File: iiwa_fri_description/urdf/iiwa7.xacro (robot description, xacro)
@@ -2,9 +2,9 @@
 <robot xmlns:xacro="http://www.ros.org/wiki/xacro">
   <!-- Import all Gazebo-customization elements, including Gazebo colors -->
-  <xacro:include filename="$(find iiwa_description)/urdf/iiwa.gazebo.xacro" />
+  <xacro:include filename="$(find iiwa_fri_description)/urdf/iiwa.gazebo.xacro" />
   <!-- Import Transmissions -->
-  <xacro:include filename="$(find iiwa_description)/urdf/iiwa.transmission.xacro" />
+  <xacro:include filename="$(find iiwa_fri_description)/urdf/iiwa.transmission.xacro" />
   <!-- Include Utilities -->
-  <xacro:include filename="$(find iiwa_description)/urdf/utilities.xacro" />
+  <xacro:include filename="$(find iiwa_fri_description)/urdf/utilities.xacro" />
   <!-- some constants -->
   <xacro:property name="safety_controller_k_pos" value="100" />
@@ -29,12 +29,12 @@
         <origin xyz="0 0 0" rpy="0 0 0"/>
         <geometry>
-          <mesh filename="package://iiwa_description/meshes/iiwa7/visual/link_0.stl"/>
-        </geometry>
-        <material name="Grey"/>
-      </visual>
-      <collision>
-        <origin xyz="0 0 0" rpy="0 0 0"/>
-        <geometry>
-          <mesh filename="package://iiwa_description/meshes/iiwa7/collision/link_0.stl"/>
+          <mesh filename="package://iiwa_fri_description/meshes/iiwa7/visual/link_0.stl"/>
+        </geometry>
+        <material name="Grey"/>
+      </visual>
+      <collision>
+        <origin xyz="0 0 0" rpy="0 0 0"/>
+        <geometry>
+          <mesh filename="package://iiwa_fri_description/meshes/iiwa7/collision/link_0.stl"/>
         </geometry>
         <material name="Grey"/>
@@ -70,5 +70,5 @@
         <origin xyz="0 0 0.0075" rpy="0 0 0"/>
         <geometry>
-          <mesh filename="package://iiwa_description/meshes/iiwa7/visual/link_1.stl"/>
+          <mesh filename="package://iiwa_fri_description/meshes/iiwa7/visual/link_1.stl"/>
         </geometry>
         <material name="Orange"/>
@@ -77,5 +77,5 @@
         <origin xyz="0 0 0.0075" rpy="0 0 0"/>
         <geometry>
-          <mesh filename="package://iiwa_description/meshes/iiwa7/collision/link_1.stl"/>
+          <mesh filename="package://iiwa_fri_description/meshes/iiwa7/collision/link_1.stl"/>
         </geometry>
         <material name="Orange"/>
@@ -104,12 +104,12 @@
         <origin xyz="0 0 0" rpy="0 0 0"/>
         <geometry>
-          <mesh filename="package://iiwa_description/meshes/iiwa7/visual/link_2.stl"/>
-        </geometry>
-        <material name="Orange"/>
-      </visual>
-      <collision>
-        <origin xyz="0 0 0" rpy="0 0 0"/>
-        <geometry>
-          <mesh filename="package://iiwa_description/meshes/iiwa7/collision/link_2.stl"/>
+          <mesh filename="package://iiwa_fri_description/meshes/iiwa7/visual/link_2.stl"/>
+        </geometry>
+        <material name="Orange"/>
+      </visual>
+      <collision>
+        <origin xyz="0 0 0" rpy="0 0 0"/>
+        <geometry>
+          <mesh filename="package://iiwa_fri_description/meshes/iiwa7/collision/link_2.stl"/>
         </geometry>
         <material name="Orange"/>
@@ -138,12 +138,12 @@
         <origin xyz="0 0 -0.026" rpy="0 0 0"/>
         <geometry>
-          <mesh filename="package://iiwa_description/meshes/iiwa7/visual/link_3.stl"/>
-        </geometry>
-        <material name="Orange"/>
-      </visual>
-      <collision>
-        <origin xyz="0 0 -0.026" rpy="0 0 0"/>
-        <geometry>
-          <mesh filename="package://iiwa_description/meshes/iiwa7/collision/link_3.stl"/>
+          <mesh filename="package://iiwa_fri_description/meshes/iiwa7/visual/link_3.stl"/>
+        </geometry>
+        <material name="Orange"/>
+      </visual>
+      <collision>
+        <origin xyz="0 0 -0.026" rpy="0 0 0"/>
+        <geometry>
+          <mesh filename="package://iiwa_fri_description/meshes/iiwa7/collision/link_3.stl"/>
         </geometry>
         <material name="Orange"/>
@@ -172,12 +172,12 @@
         <origin xyz="0 0 0" rpy="0 0 0"/>
         <geometry>
-          <mesh filename="package://iiwa_description/meshes/iiwa7/visual/link_4.stl"/>
-        </geometry>
-        <material name="Orange"/>
-      </visual>
-      <collision>
-        <origin xyz="0 0 0" rpy="0 0 0"/>
-        <geometry>
-          <mesh filename="package://iiwa_description/meshes/iiwa7/collision/link_4.stl"/>
+          <mesh filename="package://iiwa_fri_description/meshes/iiwa7/visual/link_4.stl"/>
+        </geometry>
+        <material name="Orange"/>
+      </visual>
+      <collision>
+        <origin xyz="0 0 0" rpy="0 0 0"/>
+        <geometry>
+          <mesh filename="package://iiwa_fri_description/meshes/iiwa7/collision/link_4.stl"/>
         </geometry>
         <material name="Orange"/>
@@ -206,12 +206,12 @@
         <origin xyz="0 0 -0.026" rpy="0 0 0"/>
         <geometry>
-          <mesh filename="package://iiwa_description/meshes/iiwa7/visual/link_5.stl"/>
-        </geometry>
-        <material name="Orange"/>
-      </visual>
-      <collision>
-        <origin xyz="0 0 -0.026" rpy="0 0 0"/>
-        <geometry>
-          <mesh filename="package://iiwa_description/meshes/iiwa7/collision/link_5.stl"/>
+          <mesh filename="package://iiwa_fri_description/meshes/iiwa7/visual/link_5.stl"/>
+        </geometry>
+        <material name="Orange"/>
+      </visual>
+      <collision>
+        <origin xyz="0 0 -0.026" rpy="0 0 0"/>
+        <geometry>
+          <mesh filename="package://iiwa_fri_description/meshes/iiwa7/collision/link_5.stl"/>
         </geometry>
         <material name="Orange"/>
@@ -240,12 +240,12 @@
         <origin xyz="0 0 0" rpy="0 0 0"/>
         <geometry>
-          <mesh filename="package://iiwa_description/meshes/iiwa7/visual/link_6.stl"/>
-        </geometry>
-        <material name="Orange"/>
-      </visual>
-      <collision>
-        <origin xyz="0 0 0" rpy="0 0 0"/>
-        <geometry>
-          <mesh filename="package://iiwa_description/meshes/iiwa7/collision/link_6.stl"/>
+          <mesh filename="package://iiwa_fri_description/meshes/iiwa7/visual/link_6.stl"/>
+        </geometry>
+        <material name="Orange"/>
+      </visual>
+      <collision>
+        <origin xyz="0 0 0" rpy="0 0 0"/>
+        <geometry>
+          <mesh filename="package://iiwa_fri_description/meshes/iiwa7/collision/link_6.stl"/>
         </geometry>
         <material name="Orange"/>
@@ -274,5 +274,5 @@
         <origin xyz="0 0 -0.0005" rpy="0 0 0"/>
         <geometry>
-          <mesh filename="package://iiwa_description/meshes/iiwa7/visual/link_7.stl"/>
+          <mesh filename="package://iiwa_fri_description/meshes/iiwa7/visual/link_7.stl"/>
         </geometry>
         <material name="Grey"/>
@@ -281,5 +281,5 @@
         <origin xyz="0 0 -0.0005" rpy="0 0 0"/>
         <geometry>
-          <mesh filename="package://iiwa_description/meshes/iiwa7/collision/link_7.stl"/>
+          <mesh filename="package://iiwa_fri_description/meshes/iiwa7/collision/link_7.stl"/>
         </geometry>
         <material name="Grey"/>

Commit message: Dual iiwa controllers working, moveit not finding joint states

File: iiwa_fri_description/urdf/dual_iiwa.urdf.xacro (robot description, xacro)
@@ -13,8 +13,8 @@
   </gazebo>
   <xacro:iiwa7 hardware_interface="$(arg hardware_interface)" robot_name="iiwa7" parent="world">
-    <origin xyz="0 0 0" rpy="0 0 0"/>
+    <origin xyz="0.0 0.0 0.006" rpy="0.0 0.0 ${pi/2}"/>
   </xacro:iiwa7>
   <xacro:iiwa14 hardware_interface="$(arg hardware_interface)" robot_name="iiwa14" parent="world">
-    <origin xyz="0.909536 0.612165 0.00393988" rpy="-0.00276109 0.00294195 -1.56426"/>
+    <origin xyz="0.0 0.7 0.008" rpy="0.0 0.0 ${-pi/2}"/>
   </xacro:iiwa14>
 </robot>
