Commit message: starting to test individual arm running fri, need to init the iiwastate container as zeros and do checks on commanded values

File: iiwa_fri_description/urdf/iiwa14.urdf.xacro (robot description, xacro)
@@ -10,5 +10,5 @@
   <xacro:arg name="origin_rpy" default="0 0 0"/>
   <!-- Fix to world just for testing -->
-  <link name="world"/>
+  <!--<link name="world"/> -->
   <!--iiwa-->
   <xacro:iiwa14 hardware_interface="$(arg hardware_interface)" robot_name="$(arg robot_name)" parent="world">

File: iiwa_fri_description/urdf/iiwa14.xacro (robot description, xacro)
@@ -87,5 +87,5 @@
       <child link="${robot_name}_link_2"/>
       <origin xyz="0 0 0.2025" rpy="${PI / 2}   0 ${PI}"/>
-      <axis xyz="0 0 1"/>
+      <axis xyz="0 0 1"/>http://www.ros.org/wiki/xacro
       <limit lower="${-120 * PI / 180}" upper="${120 * PI / 180}"
              effort="${max_effort}" velocity="${max_velocity}" />
@@ -145,5 +145,5 @@
       </visual>
       <collision>
-        <origin xyz="0 0 0" rpy="0 0 0"/>
+        <origin xyz="0 0 0" rpy="0 0 0"/>http://www.ros.org/wiki/xacro
         <geometry>
           <mesh filename="package://iiwa_fri_description/meshes/iiwa14/collision/link_3.stl"/>
@@ -184,5 +184,5 @@
           <mesh filename="package://iiwa_fri_description/meshes/iiwa14/collision/link_4.stl"/>
         </geometry>
-        <material name="Orange"/>
+        <material name="Orange"/>http://www.ros.org/wiki/xacro
       </collision>
     </link>
@@ -211,5 +211,5 @@
         <geometry>
           <mesh filename="package://iiwa_fri_description/meshes/iiwa14/visual/link_5.stl"/>
-        </geometry>
+        </geometry>http://www.ros.org/wiki/xacro
         <material name="Orange"/>
       </visual>
@@ -258,5 +258,5 @@
     </link>
     <!-- joint between link_6 and link_7 -->
-    <joint name="${robot_name}_joint_7" type="revolute">
+    <joint name="${robot_name}_joint_7" type="revolute">http://www.ros.org/wiki/xacro
       <parent link="${robot_name}_link_6"/>
       <child link="${robot_name}_link_7"/>

Commit message: Removed startup jerk in high frequency control mode. Filled in package information Removed old dependency on iiwa_description package

File: iiwa_fri_description/urdf/iiwa14.urdf.xacro (robot description, xacro)
@@ -10,5 +10,5 @@
   <xacro:arg name="origin_rpy" default="0 0 0"/>
   <!-- Fix to world just for testing -->
-  <!--<link name="world"/> -->
+  <link name="world"/>
   <!--iiwa-->
   <xacro:iiwa14 hardware_interface="$(arg hardware_interface)" robot_name="$(arg robot_name)" parent="world">
