Commit message: Adding in support for Effort Joint Interface currently working in iiwa_control_sim within the iiwa_fri_gazebo package. Controller params need to be tuned, only working in simulation.

File: iiwa_fri_description/urdf/iiwa.gazebo.xacro (robot description, xacro)
@@ -6,5 +6,5 @@
             <plugin name="gazebo_ros_control" filename="libgazebo_ros_control.so">
                 <robotNamespace>/${robot_name}</robotNamespace>
-                <controlPeriod>0.002</controlPeriod>
+                <controlPeriod>0.001</controlPeriod>
             </plugin>
         </gazebo>

File: iiwa_fri_description/urdf/iiwa7.xacro (robot description, xacro)
@@ -11,6 +11,6 @@
   <xacro:property name="safety_controller_k_vel" value="2" />
   <xacro:property name="joint_damping" value="0.5" />
-  <xacro:property name="max_effort" value="300"/>
-  <xacro:property name="max_velocity" value="10"/>
+  <xacro:property name="max_effort" value="5000"/>
+  <xacro:property name="max_velocity" value="100"/>
   <xacro:macro name="iiwa7" params="parent hardware_interface robot_name *origin">
     <!--joint between {parent} and link_0-->

Commit message: Cleaning up the description files

File: iiwa_fri_description/urdf/iiwa.gazebo.xacro (robot description, xacro)
@@ -1,60 +1,58 @@
 <?xml version="1.0"?>
 <robot xmlns:xacro="http://www.ros.org/wiki/xacro">
-    <xacro:macro name="iiwa_gazebo" params="robot_name">
-        <!-- Load Gazebo lib and set the robot namespace -->
-        <gazebo>
-            <plugin name="gazebo_ros_control" filename="libgazebo_ros_control.so">
-                <robotNamespace>/${robot_name}</robotNamespace>
-                <controlPeriod>0.001</controlPeriod>
-            </plugin>
-        </gazebo>
-        <!-- Link0 -->
-        <gazebo reference="${robot_name}_link_0">
-            <material>Gazebo/Grey</material>
-            <mu1>0.2</mu1>
-            <mu2>0.2</mu2>
-        </gazebo>
-        <!-- Link1 -->
-        <gazebo reference="${robot_name}_link_1">
-            <material>Gazebo/Orange</material>
-            <mu1>0.2</mu1>
-            <mu2>0.2</mu2>
-        </gazebo>
-        <!-- Link2 -->
-        <gazebo reference="${robot_name}_link_2">
-            <material>Gazebo/Orange</material>
-            <mu1>0.2</mu1>
-            <mu2>0.2</mu2>
-        </gazebo>
-        <!-- Link3 -->
-        <gazebo reference="${robot_name}_link_3">
-            <material>Gazebo/Orange</material>
-            <mu1>0.2</mu1>
-            <mu2>0.2</mu2>
-        </gazebo>
-        <!-- Link4 -->
-        <gazebo reference="${robot_name}_link_4">
-            <material>Gazebo/Orange</material>
-            <mu1>0.2</mu1>
-            <mu2>0.2</mu2>
-        </gazebo>
-        <!-- Link5 -->
-        <gazebo reference="${robot_name}_link_5">
-            <material>Gazebo/Orange</material>
-            <mu1>0.2</mu1>
-            <mu2>0.2</mu2>
-        </gazebo>
-        <!-- Link6 -->
-        <gazebo reference="${robot_name}_link_6">
-            <material>Gazebo/Orange</material>
-            <mu1>0.2</mu1>
-            <mu2>0.2</mu2>
-        </gazebo>
-        <!-- Link7 -->
-        <gazebo reference="${robot_name}_link_7">
-            <material>Gazebo/Grey</material>
-            <mu1>0.2</mu1>
-            <mu2>0.2</mu2>
-        </gazebo>
-    </xacro:macro>
+  <xacro:macro name="iiwa_gazebo" params="robot_name">
+    <gazebo>
+      <plugin name="gazebo_ros_control" filename="libgazebo_ros_control.so">
+        <robotNamespace>/${robot_name}</robotNamespace>
+      </plugin>
+    </gazebo>
+    <!-- Link0 -->
+    <gazebo reference="${robot_name}_link_0">
+      <material>Gazebo/Grey</material>
+      <mu1>0.2</mu1>
+      <mu2>0.2</mu2>
+    </gazebo>
+    <!-- Link1 -->
+    <gazebo reference="${robot_name}_link_1">
+      <material>Gazebo/Orange</material>
+      <mu1>0.2</mu1>
+      <mu2>0.2</mu2>
+    </gazebo>
+    <!-- Link2 -->
+    <gazebo reference="${robot_name}_link_2">
+      <material>Gazebo/Orange</material>
+      <mu1>0.2</mu1>
+      <mu2>0.2</mu2>
+    </gazebo>
+    <!-- Link3 -->
+    <gazebo reference="${robot_name}_link_3">
+      <material>Gazebo/Orange</material>
+      <mu1>0.2</mu1>
+      <mu2>0.2</mu2>
+    </gazebo>
+    <!-- Link4 -->
+    <gazebo reference="${robot_name}_link_4">
+      <material>Gazebo/Orange</material>
+      <mu1>0.2</mu1>
+      <mu2>0.2</mu2>
+    </gazebo>
+    <!-- Link5 -->
+    <gazebo reference="${robot_name}_link_5">
+      <material>Gazebo/Orange</material>
+      <mu1>0.2</mu1>
+      <mu2>0.2</mu2>
+    </gazebo>
+    <!-- Link6 -->
+    <gazebo reference="${robot_name}_link_6">
+      <material>Gazebo/Orange</material>
+      <mu1>0.2</mu1>
+      <mu2>0.2</mu2>
+    </gazebo>
+    <!-- Link7 -->
+    <gazebo reference="${robot_name}_link_7">
+      <material>Gazebo/Grey</material>
+      <mu1>0.2</mu1>
+      <mu2>0.2</mu2>
+    </gazebo>
+  </xacro:macro>
 </robot>

File: iiwa_fri_description/urdf/iiwa.transmission.xacro (robot description, xacro)
@@ -1,7 +1,6 @@
 <?xml version="1.0"?>
 <robot xmlns:xacro="http://www.ros.org/wiki/xacro">
-  <xacro:macro name="iiwa_transmission" params="hardware_interface">
+  <xacro:macro name="iiwa_transmission" params="hardware_interface robot_name">
     <transmission name="${robot_name}_tran_1">
-      <robotNamespace>/${robot_name}</robotNamespace>
       <type>transmission_interface/SimpleTransmission</type>
       <joint name="${robot_name}_joint_1">
@@ -14,5 +13,4 @@
     </transmission>
     <transmission name="${robot_name}_tran_2">
-      <robotNamespace>/${robot_name}</robotNamespace>
       <type>transmission_interface/SimpleTransmission</type>
       <joint name="${robot_name}_joint_2">
@@ -25,5 +23,4 @@
     </transmission>
     <transmission name="${robot_name}_tran_3">
-      <robotNamespace>/${robot_name}</robotNamespace>
       <type>transmission_interface/SimpleTransmission</type>
       <joint name="${robot_name}_joint_3">
@@ -36,5 +33,4 @@
     </transmission>
     <transmission name="${robot_name}_tran_4">
-      <robotNamespace>/${robot_name}</robotNamespace>
       <type>transmission_interface/SimpleTransmission</type>
       <joint name="${robot_name}_joint_4">
@@ -47,5 +43,4 @@
     </transmission>
     <transmission name="${robot_name}_tran_5">
-      <robotNamespace>/${robot_name}</robotNamespace>
       <type>transmission_interface/SimpleTransmission</type>
       <joint name="${robot_name}_joint_5">
@@ -58,5 +53,4 @@
     </transmission>
     <transmission name="${robot_name}_tran_6">
-      <robotNamespace>/${robot_name}</robotNamespace>
       <type>transmission_interface/SimpleTransmission</type>
       <joint name="${robot_name}_joint_6">
@@ -69,5 +63,4 @@
     </transmission>
     <transmission name="${robot_name}_tran_7">
-      <robotNamespace>/${robot_name}</robotNamespace>
       <type>transmission_interface/SimpleTransmission</type>
       <joint name="${robot_name}_joint_7">

File: iiwa_fri_description/urdf/iiwa14.xacro (robot description, xacro)
@@ -13,11 +13,5 @@
   <xacro:property name="max_effort" value="300"/>
   <xacro:property name="max_velocity" value="10"/>
-  <xacro:macro name="iiwa14" params="parent hardware_interface robot_name *origin">
-    <!--joint between {parent} and link_0-->
-    <joint name="${parent}_${robot_name}_joint" type="fixed">
-      <xacro:insert_block name="origin"/>
-      <parent link="${parent}"/>
-      <child link="${robot_name}_link_0"/>
-    </joint>
+  <xacro:macro name="iiwa14" params="hardware_interface robot_name">
     <link name="${robot_name}_link_0">
       <inertial>
@@ -87,5 +81,5 @@
       <child link="${robot_name}_link_2"/>
       <origin xyz="0 0 0.2025" rpy="${PI / 2}   0 ${PI}"/>
-      <axis xyz="0 0 1"/>http://www.ros.org/wiki/xacro
+      <axis xyz="0 0 1"/>
       <limit lower="${-120 * PI / 180}" upper="${120 * PI / 180}"
              effort="${max_effort}" velocity="${max_velocity}" />
@@ -145,5 +139,5 @@
       </visual>
       <collision>
-        <origin xyz="0 0 0" rpy="0 0 0"/>http://www.ros.org/wiki/xacro
+        <origin xyz="0 0 0" rpy="0 0 0"/>
         <geometry>
           <mesh filename="package://iiwa_fri_description/meshes/iiwa14/collision/link_3.stl"/>
@@ -184,5 +178,5 @@
           <mesh filename="package://iiwa_fri_description/meshes/iiwa14/collision/link_4.stl"/>
         </geometry>
-        <material name="Orange"/>http://www.ros.org/wiki/xacro
+        <material name="Orange"/>
       </collision>
     </link>
@@ -211,5 +205,5 @@
         <geometry>
           <mesh filename="package://iiwa_fri_description/meshes/iiwa14/visual/link_5.stl"/>
-        </geometry>http://www.ros.org/wiki/xacro
+        </geometry>
         <material name="Orange"/>
       </visual>
@@ -258,5 +252,5 @@
     </link>
     <!-- joint between link_6 and link_7 -->
-    <joint name="${robot_name}_joint_7" type="revolute">http://www.ros.org/wiki/xacro
+    <joint name="${robot_name}_joint_7" type="revolute">
       <parent link="${robot_name}_link_6"/>
       <child link="${robot_name}_link_7"/>
@@ -301,5 +295,5 @@
     <!--Extensions -->
     <xacro:iiwa_gazebo robot_name="${robot_name}" />
-    <xacro:iiwa_transmission hardware_interface="${hardware_interface}"/>
+    <xacro:iiwa_transmission hardware_interface="${hardware_interface}" robot_name="${robot_name}"/>
   </xacro:macro>
 </robot>

File: iiwa_fri_description/urdf/iiwa7.xacro (robot description, xacro)
@@ -11,13 +11,7 @@
   <xacro:property name="safety_controller_k_vel" value="2" />
   <xacro:property name="joint_damping" value="0.5" />
-  <xacro:property name="max_effort" value="5000"/>
-  <xacro:property name="max_velocity" value="100"/>
-  <xacro:macro name="iiwa7" params="parent hardware_interface robot_name *origin">
-    <!--joint between {parent} and link_0-->
-    <joint name="${parent}_${robot_name}_joint" type="fixed">
-      <xacro:insert_block name="origin"/>
-      <parent link="${parent}"/>
-      <child link="${robot_name}_link_0"/>
-    </joint>
+  <xacro:property name="max_effort" value="300"/>
+  <xacro:property name="max_velocity" value="10"/>
+  <xacro:macro name="iiwa7" params="hardware_interface robot_name">
     <link name="${robot_name}_link_0">
       <inertial>
