Commit message: Updated iiwa7 xacro to use beta flange

File: iiwa_fri_description/urdf/iiwa7.xacro (robot description, xacro)
@@ -2,9 +2,9 @@
 <robot xmlns:xacro="http://www.ros.org/wiki/xacro">
   <!-- Import all Gazebo-customization elements, including Gazebo colors -->
-  <xacro:include filename="$(find iiwa_fri_description)/urdf/iiwa.gazebo.xacro" />
+  <xacro:include filename="$(find sat_iiwa_description)/urdf/iiwa.gazebo.xacro" />
   <!-- Import Transmissions -->
-  <xacro:include filename="$(find iiwa_fri_description)/urdf/iiwa.transmission.xacro" />
+  <xacro:include filename="$(find sat_iiwa_description)/urdf/iiwa.transmission.xacro" />
   <!-- Include Utilities -->
-  <xacro:include filename="$(find iiwa_fri_description)/urdf/utilities.xacro" />
+  <xacro:include filename="$(find sat_iiwa_description)/urdf/utilities.xacro" />
   <!-- some constants -->
   <xacro:property name="safety_controller_k_pos" value="100" />
@@ -23,12 +23,12 @@
         <origin xyz="0 0 0" rpy="0 0 0"/>
         <geometry>
-          <mesh filename="package://iiwa_fri_description/meshes/iiwa7/visual/link_0.stl"/>
-        </geometry>
-        <material name="Grey"/>
-      </visual>
-      <collision>
-        <origin xyz="0 0 0" rpy="0 0 0"/>
-        <geometry>
-          <mesh filename="package://iiwa_fri_description/meshes/iiwa7/collision/link_0.stl"/>
+          <mesh filename="package://sat_iiwa_description/meshes/iiwa7/visual/link_0.stl"/>
+        </geometry>
+        <material name="Grey"/>
+      </visual>
+      <collision>
+        <origin xyz="0 0 0" rpy="0 0 0"/>
+        <geometry>
+          <mesh filename="package://sat_iiwa_description/meshes/iiwa7/collision/link_0.stl"/>
         </geometry>
         <material name="Grey"/>
@@ -64,5 +64,5 @@
         <origin xyz="0 0 0.0075" rpy="0 0 0"/>
         <geometry>
-          <mesh filename="package://iiwa_fri_description/meshes/iiwa7/visual/link_1.stl"/>
+          <mesh filename="package://sat_iiwa_description/meshes/iiwa7/visual/link_1.stl"/>
         </geometry>
         <material name="Orange"/>
@@ -71,5 +71,5 @@
         <origin xyz="0 0 0.0075" rpy="0 0 0"/>
         <geometry>
-          <mesh filename="package://iiwa_fri_description/meshes/iiwa7/collision/link_1.stl"/>
+          <mesh filename="package://sat_iiwa_description/meshes/iiwa7/collision/link_1.stl"/>
         </geometry>
         <material name="Orange"/>
@@ -98,12 +98,12 @@
         <origin xyz="0 0 0" rpy="0 0 0"/>
         <geometry>
-          <mesh filename="package://iiwa_fri_description/meshes/iiwa7/visual/link_2.stl"/>
-        </geometry>
-        <material name="Orange"/>
-      </visual>
-      <collision>
-        <origin xyz="0 0 0" rpy="0 0 0"/>
-        <geometry>
-          <mesh filename="package://iiwa_fri_description/meshes/iiwa7/collision/link_2.stl"/>
+          <mesh filename="package://sat_iiwa_description/meshes/iiwa7/visual/link_2.stl"/>
+        </geometry>
+        <material name="Orange"/>
+      </visual>
+      <collision>
+        <origin xyz="0 0 0" rpy="0 0 0"/>
+        <geometry>
+          <mesh filename="package://sat_iiwa_description/meshes/iiwa7/collision/link_2.stl"/>
         </geometry>
         <material name="Orange"/>
@@ -132,12 +132,12 @@
         <origin xyz="0 0 -0.026" rpy="0 0 0"/>
         <geometry>
-          <mesh filename="package://iiwa_fri_description/meshes/iiwa7/visual/link_3.stl"/>
-        </geometry>
-        <material name="Orange"/>
-      </visual>
-      <collision>
-        <origin xyz="0 0 -0.026" rpy="0 0 0"/>
-        <geometry>
-          <mesh filename="package://iiwa_fri_description/meshes/iiwa7/collision/link_3.stl"/>
+          <mesh filename="package://sat_iiwa_description/meshes/iiwa7/visual/link_3.stl"/>
+        </geometry>
+        <material name="Orange"/>
+      </visual>
+      <collision>
+        <origin xyz="0 0 -0.026" rpy="0 0 0"/>
+        <geometry>
+          <mesh filename="package://sat_iiwa_description/meshes/iiwa7/collision/link_3.stl"/>
         </geometry>
         <material name="Orange"/>
@@ -166,12 +166,12 @@
         <origin xyz="0 0 0" rpy="0 0 0"/>
         <geometry>
-          <mesh filename="package://iiwa_fri_description/meshes/iiwa7/visual/link_4.stl"/>
-        </geometry>
-        <material name="Orange"/>
-      </visual>
-      <collision>
-        <origin xyz="0 0 0" rpy="0 0 0"/>
-        <geometry>
-          <mesh filename="package://iiwa_fri_description/meshes/iiwa7/collision/link_4.stl"/>
+          <mesh filename="package://sat_iiwa_description/meshes/iiwa7/visual/link_4.stl"/>
+        </geometry>
+        <material name="Orange"/>
+      </visual>
+      <collision>
+        <origin xyz="0 0 0" rpy="0 0 0"/>
+        <geometry>
+          <mesh filename="package://sat_iiwa_description/meshes/iiwa7/collision/link_4.stl"/>
         </geometry>
         <material name="Orange"/>
@@ -200,12 +200,12 @@
         <origin xyz="0 0 -0.026" rpy="0 0 0"/>
         <geometry>
-          <mesh filename="package://iiwa_fri_description/meshes/iiwa7/visual/link_5.stl"/>
-        </geometry>
-        <material name="Orange"/>
-      </visual>
-      <collision>
-        <origin xyz="0 0 -0.026" rpy="0 0 0"/>
-        <geometry>
-          <mesh filename="package://iiwa_fri_description/meshes/iiwa7/collision/link_5.stl"/>
+          <mesh filename="package://sat_iiwa_description/meshes/iiwa7/visual/link_5.stl"/>
+        </geometry>
+        <material name="Orange"/>
+      </visual>
+      <collision>
+        <origin xyz="0 0 -0.026" rpy="0 0 0"/>
+        <geometry>
+          <mesh filename="package://sat_iiwa_description/meshes/iiwa7/collision/link_5.stl"/>
         </geometry>
         <material name="Orange"/>
@@ -234,12 +234,12 @@
         <origin xyz="0 0 0" rpy="0 0 0"/>
         <geometry>
-          <mesh filename="package://iiwa_fri_description/meshes/iiwa7/visual/link_6.stl"/>
-        </geometry>
-        <material name="Orange"/>
-      </visual>
-      <collision>
-        <origin xyz="0 0 0" rpy="0 0 0"/>
-        <geometry>
-          <mesh filename="package://iiwa_fri_description/meshes/iiwa7/collision/link_6.stl"/>
+          <mesh filename="package://sat_iiwa_description/meshes/iiwa7/visual/link_6.stl"/>
+        </geometry>
+        <material name="Orange"/>
+      </visual>
+      <collision>
+        <origin xyz="0 0 0" rpy="0 0 0"/>
+        <geometry>
+          <mesh filename="package://sat_iiwa_description/meshes/iiwa7/collision/link_6.stl"/>
         </geometry>
         <material name="Orange"/>
@@ -268,5 +268,5 @@
         <origin xyz="0 0 -0.0005" rpy="0 0 0"/>
         <geometry>
-          <mesh filename="package://iiwa_fri_description/meshes/iiwa7/visual/link_7.stl"/>
+          <mesh filename="package://sat_iiwa_description/meshes/iiwa7/visual/link_7.stl"/>
         </geometry>
         <material name="Grey"/>
@@ -275,5 +275,5 @@
         <origin xyz="0 0 -0.0005" rpy="0 0 0"/>
         <geometry>
-          <mesh filename="package://iiwa_fri_description/meshes/iiwa7/collision/link_7.stl"/>
+          <mesh filename="package://sat_iiwa_description/meshes/iiwa7/collision/link_7.stl"/>
         </geometry>
         <material name="Grey"/>
@@ -283,5 +283,5 @@
       <parent link="${robot_name}_link_7"/>
       <child link="${robot_name}_link_ee"/>
-      <origin xyz="0 0 0.045" rpy="0 0 0"/>
+      <origin xyz="0 0 0.0599" rpy="0 0 0"/> <!--iiwa light beta flange) -->
     </joint>
     <link name="${robot_name}_link_ee">
