Commit message: fixed error in iiwa7 looking for meshes from another package

File: iiwa_fri_description/urdf/example_iiwa7.urdf.xacro (robot description, xacro)
@@ -1,24 +1,16 @@
 <?xml version="1.0"?>
-<robot xmlns:xacro="http://www.ros.org/wiki/xacro" name="im_iiwa">
+<robot xmlns:xacro="http://www.ros.org/wiki/xacro" name="iiwa">
     <xacro:arg name="hardware_interface" default="PositionJointInterface"/>
     <xacro:arg name="initial_z" default="0.0"/>
     <link name="world"/>
     <xacro:include filename="$(find iiwa_fri_description)/urdf/iiwa14.xacro"/>
-    <xacro:arg name="eye_robot_name" default="im_iiwa"/>
+    <xacro:arg name="robot_name" default="iiwa"/>
     <xacro:arg name="hardware_interface" default="PositionJointInterface"/>
-    <joint name="$(arg eye_robot_name)_world_joint" type="fixed">
+    <joint name="$(arg robot_name)_world_joint" type="fixed">
         <parent link="world"/>
-        <child link="$(arg eye_robot_name)_link_0"/>
+        <child link="$(arg robot_name)_link_0"/>
         <origin xyz="0.0 0.0 0.006" rpy="0.0 0.0 ${pi/2}"/>
     </joint>
-    <xacro:iiwa14 hardware_interface="$(arg hardware_interface)" robot_name="$(arg eye_robot_name)">
+    <xacro:iiwa14 hardware_interface="$(arg hardware_interface)" robot_name="$(arg robot_name)">
     </xacro:iiwa14>
-    <!--
-    <xacro:include filename="$(find sat_description)/sensors/kinect.urdf.xacro"/>
-    <joint name="$(arg eye_robot_name)_ee_to_eye" type="fixed">
-        <parent link="$(arg eye_robot_name)_link_ee"/>
-        <child link="camera_link"/>
-		<origin xyz="0.012 0.0 0.1" rpy="${0.0} ${-pi/2} ${0.0}"/>
-    </joint>
-    -->
 </robot>

File: iiwa_fri_description/urdf/iiwa7.xacro (robot description, xacro)
@@ -2,9 +2,9 @@
 <robot xmlns:xacro="http://www.ros.org/wiki/xacro">
   <!-- Import all Gazebo-customization elements, including Gazebo colors -->
-  <xacro:include filename="$(find sat_iiwa_description)/urdf/iiwa.gazebo.xacro" />
+  <xacro:include filename="$(find iiwa_fri_description)/urdf/iiwa.gazebo.xacro" />
   <!-- Import Transmissions -->
-  <xacro:include filename="$(find sat_iiwa_description)/urdf/iiwa.transmission.xacro" />
+  <xacro:include filename="$(find iiwa_fri_description)/urdf/iiwa.transmission.xacro" />
   <!-- Include Utilities -->
-  <xacro:include filename="$(find sat_iiwa_description)/urdf/utilities.xacro" />
+  <xacro:include filename="$(find iiwa_fri_description)/urdf/utilities.xacro" />
   <!-- some constants -->
   <xacro:property name="safety_controller_k_pos" value="100" />
@@ -23,12 +23,12 @@
         <origin xyz="0 0 0" rpy="0 0 0"/>
         <geometry>
-          <mesh filename="package://sat_iiwa_description/meshes/iiwa7/visual/link_0.stl"/>
-        </geometry>
-        <material name="Grey"/>
-      </visual>
-      <collision>
-        <origin xyz="0 0 0" rpy="0 0 0"/>
-        <geometry>
-          <mesh filename="package://sat_iiwa_description/meshes/iiwa7/collision/link_0.stl"/>
+          <mesh filename="package://iiwa_fri_description/meshes/iiwa7/visual/link_0.stl"/>
+        </geometry>
+        <material name="Grey"/>
+      </visual>
+      <collision>
+        <origin xyz="0 0 0" rpy="0 0 0"/>
+        <geometry>
+          <mesh filename="package://iiwa_fri_description/meshes/iiwa7/collision/link_0.stl"/>
         </geometry>
         <material name="Grey"/>
@@ -64,5 +64,5 @@
         <origin xyz="0 0 0.0075" rpy="0 0 0"/>
         <geometry>
-          <mesh filename="package://sat_iiwa_description/meshes/iiwa7/visual/link_1.stl"/>
+          <mesh filename="package://iiwa_fri_description/meshes/iiwa7/visual/link_1.stl"/>
         </geometry>
         <material name="Orange"/>
@@ -71,5 +71,5 @@
         <origin xyz="0 0 0.0075" rpy="0 0 0"/>
         <geometry>
-          <mesh filename="package://sat_iiwa_description/meshes/iiwa7/collision/link_1.stl"/>
+          <mesh filename="package://iiwa_fri_description/meshes/iiwa7/collision/link_1.stl"/>
         </geometry>
         <material name="Orange"/>
@@ -98,12 +98,12 @@
         <origin xyz="0 0 0" rpy="0 0 0"/>
         <geometry>
-          <mesh filename="package://sat_iiwa_description/meshes/iiwa7/visual/link_2.stl"/>
-        </geometry>
-        <material name="Orange"/>
-      </visual>
-      <collision>
-        <origin xyz="0 0 0" rpy="0 0 0"/>
-        <geometry>
-          <mesh filename="package://sat_iiwa_description/meshes/iiwa7/collision/link_2.stl"/>
+          <mesh filename="package://iiwa_fri_description/meshes/iiwa7/visual/link_2.stl"/>
+        </geometry>
+        <material name="Orange"/>
+      </visual>
+      <collision>
+        <origin xyz="0 0 0" rpy="0 0 0"/>
+        <geometry>
+          <mesh filename="package://iiwa_fri_description/meshes/iiwa7/collision/link_2.stl"/>
         </geometry>
         <material name="Orange"/>
@@ -132,12 +132,12 @@
         <origin xyz="0 0 -0.026" rpy="0 0 0"/>
         <geometry>
-          <mesh filename="package://sat_iiwa_description/meshes/iiwa7/visual/link_3.stl"/>
-        </geometry>
-        <material name="Orange"/>
-      </visual>
-      <collision>
-        <origin xyz="0 0 -0.026" rpy="0 0 0"/>
-        <geometry>
-          <mesh filename="package://sat_iiwa_description/meshes/iiwa7/collision/link_3.stl"/>
+          <mesh filename="package://iiwa_fri_description/meshes/iiwa7/visual/link_3.stl"/>
+        </geometry>
+        <material name="Orange"/>
+      </visual>
+      <collision>
+        <origin xyz="0 0 -0.026" rpy="0 0 0"/>
+        <geometry>
+          <mesh filename="package://iiwa_fri_description/meshes/iiwa7/collision/link_3.stl"/>
         </geometry>
         <material name="Orange"/>
@@ -166,12 +166,12 @@
         <origin xyz="0 0 0" rpy="0 0 0"/>
         <geometry>
-          <mesh filename="package://sat_iiwa_description/meshes/iiwa7/visual/link_4.stl"/>
-        </geometry>
-        <material name="Orange"/>
-      </visual>
-      <collision>
-        <origin xyz="0 0 0" rpy="0 0 0"/>
-        <geometry>
-          <mesh filename="package://sat_iiwa_description/meshes/iiwa7/collision/link_4.stl"/>
+          <mesh filename="package://iiwa_fri_description/meshes/iiwa7/visual/link_4.stl"/>
+        </geometry>
+        <material name="Orange"/>
+      </visual>
+      <collision>
+        <origin xyz="0 0 0" rpy="0 0 0"/>
+        <geometry>
+          <mesh filename="package://iiwa_fri_description/meshes/iiwa7/collision/link_4.stl"/>
         </geometry>
         <material name="Orange"/>
@@ -200,12 +200,12 @@
         <origin xyz="0 0 -0.026" rpy="0 0 0"/>
         <geometry>
-          <mesh filename="package://sat_iiwa_description/meshes/iiwa7/visual/link_5.stl"/>
-        </geometry>
-        <material name="Orange"/>
-      </visual>
-      <collision>
-        <origin xyz="0 0 -0.026" rpy="0 0 0"/>
-        <geometry>
-          <mesh filename="package://sat_iiwa_description/meshes/iiwa7/collision/link_5.stl"/>
+          <mesh filename="package://iiwa_fri_description/meshes/iiwa7/visual/link_5.stl"/>
+        </geometry>
+        <material name="Orange"/>
+      </visual>
+      <collision>
+        <origin xyz="0 0 -0.026" rpy="0 0 0"/>
+        <geometry>
+          <mesh filename="package://iiwa_fri_description/meshes/iiwa7/collision/link_5.stl"/>
         </geometry>
         <material name="Orange"/>
@@ -234,12 +234,12 @@
         <origin xyz="0 0 0" rpy="0 0 0"/>
         <geometry>
-          <mesh filename="package://sat_iiwa_description/meshes/iiwa7/visual/link_6.stl"/>
-        </geometry>
-        <material name="Orange"/>
-      </visual>
-      <collision>
-        <origin xyz="0 0 0" rpy="0 0 0"/>
-        <geometry>
-          <mesh filename="package://sat_iiwa_description/meshes/iiwa7/collision/link_6.stl"/>
+          <mesh filename="package://iiwa_fri_description/meshes/iiwa7/visual/link_6.stl"/>
+        </geometry>
+        <material name="Orange"/>
+      </visual>
+      <collision>
+        <origin xyz="0 0 0" rpy="0 0 0"/>
+        <geometry>
+          <mesh filename="package://iiwa_fri_description/meshes/iiwa7/collision/link_6.stl"/>
         </geometry>
         <material name="Orange"/>
@@ -268,5 +268,5 @@
         <origin xyz="0 0 -0.0005" rpy="0 0 0"/>
         <geometry>
-          <mesh filename="package://sat_iiwa_description/meshes/iiwa7/visual/link_7.stl"/>
+          <mesh filename="package://iiwa_fri_description/meshes/iiwa7/visual/link_7.stl"/>
         </geometry>
         <material name="Grey"/>
@@ -275,5 +275,5 @@
         <origin xyz="0 0 -0.0005" rpy="0 0 0"/>
         <geometry>
-          <mesh filename="package://sat_iiwa_description/meshes/iiwa7/collision/link_7.stl"/>
+          <mesh filename="package://iiwa_fri_description/meshes/iiwa7/collision/link_7.stl"/>
         </geometry>
         <material name="Grey"/>
