Commit message: Now logging last commanded position in degress and the joint limits of the urdfs has been reduced by 1 degree each

File: iiwa_fri_description/urdf/iiwa14.xacro (robot description, xacro)
@@ -47,5 +47,5 @@
       <origin xyz="0 0 0.1575" rpy="0 0 0"/>
       <axis xyz="0 0 1"/>
-      <limit lower="${-170 * PI / 180}" upper="${170 * PI / 180}"
+      <limit lower="${-169 * PI / 180}" upper="${169 * PI / 180}"
              effort="${max_effort}" velocity="${max_velocity}" />
       <safety_controller soft_lower_limit="${-168 * PI / 180}"
@@ -82,5 +82,5 @@
       <origin xyz="0 0 0.2025" rpy="${PI / 2}   0 ${PI}"/>
       <axis xyz="0 0 1"/>
-      <limit lower="${-120 * PI / 180}" upper="${120 * PI / 180}"
+      <limit lower="${-119 * PI / 180}" upper="${119 * PI / 180}"
              effort="${max_effort}" velocity="${max_velocity}" />
       <safety_controller soft_lower_limit="${-118 * PI / 180}"
@@ -117,5 +117,5 @@
       <origin xyz="0 0.2045 0" rpy="${PI / 2} 0 ${PI}"/>
       <axis xyz="0 0 1"/>
-      <limit lower="${-170 * PI / 180}" upper="${170 * PI / 180}"
+      <limit lower="${-169 * PI / 180}" upper="${169 * PI / 180}"
              effort="${max_effort}" velocity="${max_velocity}" />
       <safety_controller soft_lower_limit="${-168 * PI / 180}"
@@ -152,5 +152,5 @@
       <origin xyz="0 0 0.2155" rpy="${PI / 2} 0 0"/>
       <axis xyz="0 0 1"/>
-      <limit lower="${-120 * PI / 180}" upper="${120 * PI / 180}"
+      <limit lower="${-119 * PI / 180}" upper="${119 * PI / 180}"
              effort="${max_effort}" velocity="${max_velocity}" />
       <safety_controller soft_lower_limit="${-118 * PI / 180}"
@@ -187,5 +187,5 @@
       <origin xyz="0 0.1845 0" rpy="${-PI / 2} ${PI} 0"/>
       <axis xyz="0 0 1"/>
-      <limit lower="${-170 * PI / 180}" upper="${170 * PI / 180}"
+      <limit lower="${-169 * PI / 180}" upper="${169 * PI / 180}"
              effort="${max_effort}" velocity="${max_velocity}" />
       <safety_controller soft_lower_limit="${-168 * PI / 180}"
@@ -222,5 +222,5 @@
       <origin xyz="0 0 0.2155" rpy="${PI / 2} 0 0"/>
       <axis xyz="0 0 1"/>
-      <limit lower="${-120 * PI / 180}" upper="${120 * PI / 180}"
+      <limit lower="${-119 * PI / 180}" upper="${119 * PI / 180}"
              effort="${max_effort}" velocity="${max_velocity}" />
       <safety_controller soft_lower_limit="${-118 * PI / 180}"
@@ -257,5 +257,5 @@
       <origin xyz="0 0.081 0" rpy="${- PI / 2} ${PI} 0"/>
       <axis xyz="0 0 1"/>
-      <limit lower="${-175 * PI / 180}" upper="${175 * PI / 180}"
+      <limit lower="${-174 * PI / 180}" upper="${174 * PI / 180}"
              effort="${max_effort}" velocity="${max_velocity}" />
       <safety_controller soft_lower_limit="${-173 * PI / 180}"

Commit message: Soft limits are actually being loaded properly now and the iiwa hardware velocity limits have been put into the urdf

File: iiwa_fri_description/urdf/iiwa14.xacro (robot description, xacro)
@@ -8,6 +8,6 @@
   <xacro:include filename="$(find iiwa_fri_description)/urdf/utilities.xacro" />
   <!-- some constants -->
-  <xacro:property name="safety_controller_k_pos" value="100" />
-  <xacro:property name="safety_controller_k_vel" value="2" />
+  <xacro:property name="safety_controller_k_pos" value="1" />
+  <xacro:property name="safety_controller_k_vel" value="1" />
   <xacro:property name="joint_damping" value="0.5" />
   <xacro:property name="max_effort" value="300"/>
@@ -48,7 +48,7 @@
       <axis xyz="0 0 1"/>
       <limit lower="${-169 * PI / 180}" upper="${169 * PI / 180}"
-             effort="${max_effort}" velocity="${max_velocity}" />
-      <safety_controller soft_lower_limit="${-168 * PI / 180}"
-                         soft_upper_limit="${168 * PI / 180}"
+             effort="${max_effort}" velocity="{85 * PI / 180}" />
+      <safety_controller soft_lower_limit="${-169 * PI / 180}"
+                         soft_upper_limit="${169 * PI / 180}"
                          k_position="${safety_controller_k_pos}"
                          k_velocity="${safety_controller_k_vel}"/>
@@ -83,7 +83,7 @@
       <axis xyz="0 0 1"/>
       <limit lower="${-119 * PI / 180}" upper="${119 * PI / 180}"
-             effort="${max_effort}" velocity="${max_velocity}" />
-      <safety_controller soft_lower_limit="${-118 * PI / 180}"
-                         soft_upper_limit="${118 * PI / 180}"
+             effort="${max_effort}" velocity="{85 * PI / 180}" />
+      <safety_controller soft_lower_limit="${-119 * PI / 180}"
+                         soft_upper_limit="${119 * PI / 180}"
                          k_position="${safety_controller_k_pos}"
                          k_velocity="${safety_controller_k_vel}"/>
@@ -118,7 +118,7 @@
       <axis xyz="0 0 1"/>
       <limit lower="${-169 * PI / 180}" upper="${169 * PI / 180}"
-             effort="${max_effort}" velocity="${max_velocity}" />
-      <safety_controller soft_lower_limit="${-168 * PI / 180}"
-                         soft_upper_limit="${168 * PI / 180}"
+             effort="${max_effort}" velocity="{100 * PI / 180}" />
+      <safety_controller soft_lower_limit="${-169 * PI / 180}"
+                         soft_upper_limit="${169 * PI / 180}"
                          k_position="${safety_controller_k_pos}"
                          k_velocity="${safety_controller_k_vel}"/>
@@ -153,7 +153,7 @@
       <axis xyz="0 0 1"/>
       <limit lower="${-119 * PI / 180}" upper="${119 * PI / 180}"
-             effort="${max_effort}" velocity="${max_velocity}" />
-      <safety_controller soft_lower_limit="${-118 * PI / 180}"
-                         soft_upper_limit="${118 * PI / 180}"
+             effort="${max_effort}" velocity="{75 * PI / 180}" />
+      <safety_controller soft_lower_limit="${-119 * PI / 180}"
+                         soft_upper_limit="${119 * PI / 180}"
                          k_position="${safety_controller_k_pos}"
                          k_velocity="${safety_controller_k_vel}"/>
@@ -188,7 +188,7 @@
       <axis xyz="0 0 1"/>
       <limit lower="${-169 * PI / 180}" upper="${169 * PI / 180}"
-             effort="${max_effort}" velocity="${max_velocity}" />
-      <safety_controller soft_lower_limit="${-168 * PI / 180}"
-                         soft_upper_limit="${168 * PI / 180}"
+             effort="${max_effort}" velocity="{130 * PI / 180}" />
+      <safety_controller soft_lower_limit="${-169 * PI / 180}"
+                         soft_upper_limit="${169 * PI / 180}"
                          k_position="${safety_controller_k_pos}"
                          k_velocity="${safety_controller_k_vel}"/>
@@ -223,7 +223,7 @@
       <axis xyz="0 0 1"/>
       <limit lower="${-119 * PI / 180}" upper="${119 * PI / 180}"
-             effort="${max_effort}" velocity="${max_velocity}" />
-      <safety_controller soft_lower_limit="${-118 * PI / 180}"
-                         soft_upper_limit="${118 * PI / 180}"
+             effort="${max_effort}" velocity="{135 * PI / 180}" />
+      <safety_controller soft_lower_limit="${-119 * PI / 180}"
+                         soft_upper_limit="${119 * PI / 180}"
                          k_position="${safety_controller_k_pos}"
                          k_velocity="${safety_controller_k_vel}"/>
@@ -258,7 +258,7 @@
       <axis xyz="0 0 1"/>
       <limit lower="${-174 * PI / 180}" upper="${174 * PI / 180}"
-             effort="${max_effort}" velocity="${max_velocity}" />
-      <safety_controller soft_lower_limit="${-173 * PI / 180}"
-                         soft_upper_limit="${173 * PI / 180}"
+             effort="${max_effort}" velocity="{135 * PI / 180}" />
+      <safety_controller soft_lower_limit="${-174 * PI / 180}"
+                         soft_upper_limit="${174 * PI / 180}"
                          k_position="${safety_controller_k_pos}"
                          k_velocity="${safety_controller_k_vel}"/>

Commit message: Softlimits were too low, iiwa controller now outputs both last commanded and last known positions

File: iiwa_fri_description/urdf/iiwa14.xacro (robot description, xacro)
@@ -8,6 +8,6 @@
   <xacro:include filename="$(find iiwa_fri_description)/urdf/utilities.xacro" />
   <!-- some constants -->
-  <xacro:property name="safety_controller_k_pos" value="1" />
-  <xacro:property name="safety_controller_k_vel" value="1" />
+  <xacro:property name="safety_controller_k_pos" value="50" />
+  <xacro:property name="safety_controller_k_vel" value="2" />
   <xacro:property name="joint_damping" value="0.5" />
   <xacro:property name="max_effort" value="300"/>

Commit message: Joint limits are handled correctly now but the safety controller k position value still needs some tuning

File: iiwa_fri_description/urdf/iiwa14.xacro (robot description, xacro)
@@ -8,9 +8,8 @@
   <xacro:include filename="$(find iiwa_fri_description)/urdf/utilities.xacro" />
   <!-- some constants -->
-  <xacro:property name="safety_controller_k_pos" value="50" />
-  <xacro:property name="safety_controller_k_vel" value="2" />
+  <xacro:property name="safety_controller_k_pos" value="5" />
+  <xacro:property name="safety_controller_k_vel" value="4" />
   <xacro:property name="joint_damping" value="0.5" />
-  <xacro:property name="max_effort" value="300"/>
-  <xacro:property name="max_velocity" value="10"/>
+  <xacro:property name="max_effort" value="300"/> <!-- Should be changed to match the robots specs -->
   <xacro:macro name="iiwa14" params="hardware_interface robot_name">
     <link name="${robot_name}_link_0">

Commit message: Soft limits tuned and iiwa hardware launch file directly runs controller again.

File: iiwa_fri_description/urdf/iiwa14.xacro (robot description, xacro)
@@ -8,9 +8,8 @@
   <xacro:include filename="$(find iiwa_fri_description)/urdf/utilities.xacro" />
   <!-- some constants -->
-  <xacro:property name="safety_controller_k_pos" value="50" />
-  <xacro:property name="safety_controller_k_vel" value="2" />
-  <xacro:property name="joint_damping" value="0.5" />
-  <xacro:property name="max_effort" value="300"/>
-  <xacro:property name="max_velocity" value="10"/>
+  <xacro:property name="safety_controller_k_pos" value="10" /> <!-- This sets the velocity according the distance the soft limits, velocity = -k_pos * (pos - soft_limit) -->
+  <xacro:property name="safety_controller_k_vel" value="4" />
+  <xacro:property name="joint_damping" value="0.0" />
+  <xacro:property name="max_effort" value="300"/> <!-- Should be changed to match the robots specs -->
   <xacro:macro name="iiwa14" params="hardware_interface robot_name">
     <link name="${robot_name}_link_0">

Commit message: removed effort limit interfaces as they were causing instabilities when the joints are close to the limits

File: iiwa_fri_description/urdf/iiwa14.xacro (robot description, xacro)
@@ -9,5 +9,5 @@
   <!-- some constants -->
   <xacro:property name="safety_controller_k_pos" value="10" /> <!-- This sets the velocity according the distance the soft limits, velocity = -k_pos * (pos - soft_limit) -->
-  <xacro:property name="safety_controller_k_vel" value="4" />
+  <xacro:property name="safety_controller_k_vel" value="40" />
   <xacro:property name="joint_damping" value="0.0" />
   <xacro:property name="max_effort" value="300"/> <!-- Should be changed to match the robots specs -->
