Commit message: Enabling effort command interface

File: iiwa_fri_ros/config/iiwa.ros2_control.xacro (robot description, xacro)
@@ -1,5 +1,5 @@
 <?xml version="1.0"?>
 <robot xmlns:xacro="http://www.ros.org/wiki/xacro">
-    <xacro:macro name="iiwa_position_only" params="name
+    <xacro:macro name="iiwa_position_effort" params="name
     robot_ip robot_port">
         <ros2_control name="${name}" type="system">
@@ -14,4 +14,8 @@
                     <param name="max">{169 * PI / 180}</param>
                 </command_interface>
+                <command_interface name="effort">
+                    <param name="min">{-320}</param>
+                    <param name="max">{320}</param>
+                </command_interface>
                 <state_interface name="position"/>
                 <state_interface name="velocity"/>
@@ -22,4 +26,8 @@
                     <param name="min">{-119 * PI / 180}</param>
                     <param name="max">{119 * PI / 180}</param>
+                </command_interface>
+                <command_interface name="effort">
+                    <param name="min">{-320}</param>
+                    <param name="max">{320}</param>
                 </command_interface>
                 <state_interface name="position"/>
@@ -32,4 +40,8 @@
                     <param name="max">{169 * PI / 180}</param>
                 </command_interface>
+                <command_interface name="effort">
+                    <param name="min">{-176}</param>
+                    <param name="max">{176}</param>
+                </command_interface>
                 <state_interface name="position"/>
                 <state_interface name="velocity"/>
@@ -40,4 +52,8 @@
                     <param name="min">{-119 * PI / 180}</param>
                     <param name="max">{119 * PI / 180}</param>
+                </command_interface>
+                <command_interface name="effort">
+                    <param name="min">{-176}</param>
+                    <param name="max">{176}</param>
                 </command_interface>
                 <state_interface name="position"/>
@@ -50,4 +66,8 @@
                     <param name="max">{169 * PI / 180}</param>
                 </command_interface>
+                <command_interface name="effort">
+                    <param name="min">{-110}</param>
+                    <param name="max">{110}</param>
+                </command_interface>
                 <state_interface name="position"/>
                 <state_interface name="velocity"/>
@@ -58,4 +78,8 @@
                     <param name="min">{-119 * PI / 180}</param>
                     <param name="max">{119 * PI / 180}</param>
+                </command_interface>
+                <command_interface name="effort">
+                    <param name="min">{-40}</param>
+                    <param name="max">{40}</param>
                 </command_interface>
                 <state_interface name="position"/>
@@ -68,4 +92,8 @@
                     <param name="max">{174 * PI / 180}</param>
                 </command_interface>
+                <command_interface name="effort">
+                    <param name="min">{-40}</param>
+                    <param name="max">{40}</param>
+                </command_interface>
                 <state_interface name="position"/>
                 <state_interface name="velocity"/>
